File: lightsaber.kicad_pcb (KiCad board)
At the start: 2 copper layers, 7 parts, among them SW1 SW_Push, SW3 POWER, U1 C3 Pico

Commit message: Preliminary PCB layout
Parts:
- removed LIN1: LEDs_In, neopixel-strip:neopixel-strip
- added R1: VT93xx, OptoDevice:R_LDR_4.9x4.2mm_P2.54mm_Vertical, F.Cu at (107.5, 106.5)
- added R3: R, Resistor_SMD:R_0805_2012Metric_Pad1.20x1.40mm_HandSolder, B.Cu at (109.0, 109.5)
- SW1: value SW_Push -> Button
- SW3: moved to B.Cu
- moved SW3 94.9 mm to (90.5, 133.5), turned to 90 degrees
- moved NP1 81.8 mm to (99.5, 25.9), turned to 0 degrees
- moved BT1 67.1 mm to (95.0, 32.4), turned to -90 degrees
- moved U1 55.2 mm to (99.5, 120.9)
- moved R2 45.0 mm to (110.5, 34.5), turned to 90 degrees
- moved SW1 33.3 mm to (107.0, 59.5), turned to 90 degrees
- renumbered LOUT1 to NP1
Connections:
- BT1 pad 1: unconnected-(BT1-+-Pad1) -> +4V
- BT1 pad 2: unconnected-(BT1---Pad2) -> GND
- NP1 pad 1: unconnected-(LOUT1-VCC-Pad1) -> +4V
- NP1 pad 2: unconnected-(LOUT1-Data-Pad2) -> Neopixel
- NP1 pad 3: unconnected-(LOUT1-GND-Pad3) -> GND
- R2 pad 1: unconnected-(R2-Pad1) -> +3V3
- R2 pad 2: unconnected-(R2-Pad2) -> Poti
- R2 pad 3: unconnected-(R2-Pad3) -> GND
- SW1 pad 1: unconnected-(SW1-Pad1) -> GND
- SW1 pad 2: unconnected-(SW1-Pad2) -> Button
- SW3 pad 2: unconnected-(SW3-B-Pad2) -> +3V3
- SW3 pad 3: unconnected-(SW3-C-Pad3) -> Power
- U1 pad 1: unconnected-(U1-5V-Pad1) -> +5V
- U1 pad 10: unconnected-(U1-IO5-Pad10) -> Light
- U1 pad 11: unconnected-(U1-IO4/MOSI-Pad11) -> Button
- U1 pad 13: unconnected-(U1-IO1/SCK-Pad13) -> Poti
- U1 pad 14: unconnected-(U1-IO2-Pad14) -> Neopixel
- U1 pad 15: unconnected-(U1-IO3/VBAT-Pad15) -> +4V
- U1 pad 16: unconnected-(U1-RST/EN-Pad16) -> Power
- U1 pad 2: unconnected-(U1-GND-Pad2) -> GND
- U1 pad 9: unconnected-(U1-3V3-Pad9) -> +3V3
Routing:
- net +4V: track 0.00 -> 115.4 mm
- net GND: track 0.00 -> 112.6 mm, vias 0 -> 4
- net +3V3: track 0.00 -> 110.2 mm
- net Poti: track 0.00 -> 103.5 mm
- net Neopixel: track 0.00 -> 101.9 mm
- net Button: track 0.00 -> 84.8 mm
- net Light: track 0.00 -> 33.8 mm
- net Power: track 0.00 -> 23.0 mm
- added copper zone on B.Cu, net +3V3
- added copper zone on B.Cu, net GND
Other:
- board outline added: 31 x 112.5 mm
